File: hardware/HCV.kicad_pcb (KiCad board)
At the start: 2 copper layers, 49.5 x 40.5 mm, 33 parts, among them J1 USB_B_Micro, J2 Conn_ARM_SWD_TagConnect_TC2030, J4 Conn_01x02, SW2 SW_DIP_x02, U1 ESP32-WROOM-32U, U2 TPS562242, U3 SN65HVD232, U4 ADuM1201AR

Commit message: Updated Docu, Updated Hardware
Parts:
- removed J1: USB_B_Micro, Connector_USB:USB_C_Receptacle_Palconn_UTC16-G
- removed JP1, JP2: Jumper_2_Open, Jumper:SolderJumper-2_P1.3mm_Open_RoundedPad1.0x1.5mm
- removed R1, R2: 5R, Resistor_SMD:R_0805_2012Metric
- added C11: 100n, Capacitor_SMD:C_0603_1608Metric, F.Cu at (153.2, 101.3)
- added C12: 100n, Capacitor_SMD:C_0603_1608Metric, F.Cu at (153.2, 105.5)
- added J3: USB_C_Receptacle_PowerOnly_6P, Connector_USB:USB_C_Receptacle_GCT_USB4125-xx-x-0190_6P_TopMnt_Horizontal, F.Cu at (168.4, 109.1)
- added U5: TEA1-0505, Converter_DCDC:Converter_DCDC_TRACO_TEA1-xxxx_THT, F.Cu at (155.7, 99.6)
- SW2: value SW_DIP_x02 -> SW_DIP_x04; footprint Package_DIP:DIP-4_W7.62mm -> Package_DIP:DIP-8_W7.62mm
- U3: value SN65HVD232 -> ATA6560
- moved SW2 2.97 mm to (141.2, 111.3)
Connections:
- net +12V renamed +5V
- net +3.3VP renamed +5VP
- SW2 pad 3: GND -> /nRXONLY
- SW2 pad 4: Net-(R7-Pad1) -> unconnected-(SW2-Pad4)
- U3 pad 5: unconnected-(U3-NC-Pad5) -> /nRXONLY
- U3 pad 6: Net-(U3-CANL) -> Net-(D4-K)
- U3 pad 7: Net-(U3-CANH) -> Net-(D3-K)
- U3 pad 8: unconnected-(U3-NC-Pad8) -> GNDA
Routing:
- net GNDA: track 8.84 -> 39.6 mm, vias 7 -> 8
- net +5VP: track 15.5 -> 46.0 mm
- net /nRXONLY: track 0.00 -> 29.9 mm, vias 0 -> 2
- net +5V: track 17.8 -> 29.3 mm
- net Net-(D4-K): track 13.0 -> 18.2 mm
- net Net-(U3-CANL): track 3.37 -> 0.00 mm
- net Net-(U3-CANH): track 3.09 -> 0.00 mm
- net Net-(D3-K): track 30.4 -> 33.4 mm
- net Net-(R7-Pad1): track 6.81 -> 3.83 mm
- net GND: track 30.3 -> 32.3 mm, vias 15 -> 12
- net /OPTSW: track 23.2 -> 24.0 mm
Other:
- board text added: "embdes CAN-HCV 1.3"
- board text removed: "embdes HC-CAN 1.2"
