File: hardware/HCV.kicad_pcb (KiCad board)
At the start: 2 copper layers, 49.5 x 40.5 mm, 32 parts, among them J2 Conn_ARM_SWD_TagConnect_TC2030, J3 USB_C_Receptacle_PowerOnly_6P, J4 Conn_01x02, SW2 SW_DIP_x04, U1 ESP32-WROOM-32U, U2 TPS562242, U3 ATA6560, U4 ADuM1201AR, U5 TEA1-0505

Commit message: Update for HCV Hardware
Parts:
- removed D4: 1N4148WT, Diode_SMD:D_SOD-523
- removed R7: 120R, Resistor_SMD:R_0805_2012Metric
- removed SW2: SW_DIP_x04, Package_DIP:DIP-8_W7.62mm
- added C15: 100n, Capacitor_SMD:C_0603_1608Metric, F.Cu at (135.3, 87.3)
- added R1: 4k7, Resistor_SMD:R_0603_1608Metric, F.Cu at (130.4, 97.5)
- added SW1: SW_Push, Button_Switch_SMD:SW_SPST_EVPBF, B.Cu at (150.2, 88.5)
- C12: value 100n -> 33/16; footprint Capacitor_SMD:C_0603_1608Metric -> Capacitor_Tantalum_SMD:CP_EIA-3528-12_Kemet-T
- D3: value 1N4148WT -> PESD1CAN-UX; footprint Diode_SMD:D_SOD-523 -> Package_TO_SOT_SMD:SOT-23-3
- R8: value 520R -> 470R
- moved U5 25.1 mm to (132.4, 108.9), turned to 180 degrees
- moved C11 19.3 mm to (135.6, 109.2), turned to -90 degrees
- moved C12 17.1 mm to (136.3, 102.8), turned to -90 degrees
- moved J4 13.1 mm to (142.3, 104.9)
- moved D3 10.9 mm to (136.8, 91.8), turned to 90 degrees
- moved R8 8.74 mm to (154.7, 95.7), turned to 0 degrees
- moved U3 2.79 mm to (131.4, 92.4)
- moved C9 2.64 mm to (127.2, 93.7)
- moved C10 2.59 mm to (127.2, 90.3)
- moved J3 1.15 mm to (168.4, 110.2)
Connections:
- D3 pad 2: GNDA -> Net-(D3-C2)
- J4 pad 2: Net-(D4-K) -> Net-(D3-C2)
- R8 pad 1: Net-(U1-IO13) -> Net-(D1-A)
- R8 pad 2: Net-(D1-K) -> Net-(U1-IO15)
- U1 pad 14: /OPTSW -> /CANR
- U1 pad 16: Net-(U1-IO13) -> Net-(D1-K)
- U1 pad 23: Net-(D1-A) -> Net-(U1-IO15)
- U1 pad 28: unconnected-(U1-IO17-Pad28) -> Net-(U1-IO17)
- U3 pad 6: Net-(D4-K) -> Net-(D3-C2)
Routing:
- net +5VP: track 46.0 -> 6.44 mm
- net +5V: track 29.3 -> 57.1 mm, vias 0 -> 2
- net /nRXONLY: track 29.9 -> 2.66 mm, vias 2 -> 0
- net Net-(D3-C2): track 0.00 -> 27.0 mm, vias 0 -> 2
- net /OPTSW: track 24.0 -> 0.00 mm, vias 1 -> 0
- net Net-(D4-K): track 18.2 -> 0.00 mm, vias 1 -> 0
- net GNDA: track 39.6 -> 23.6 mm, vias 8 -> 5
- net Net-(U1-IO17): track 0.00 -> 14.8 mm, vias 0 -> 1
- net Net-(D3-C1): track 33.4 -> 20.5 mm
- net Net-(U1-IO15): track 0.00 -> 4.50 mm
- net Net-(U1-IO13): track 4.22 -> 0.00 mm
- net Net-(D1-A): track 7.10 -> 3.00 mm
- net Net-(D1-K): track 3.01 -> 7.04 mm
- net Net-(R7-Pad1): track 3.83 -> 0.00 mm
- net Net-(U3-D): track 10.2 -> 8.82 mm, vias 2 -> 0
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- added copper zone on F.Cu, net +5VP
Other:
- board text added: "embdes CAN-HCV 1.6"
- board text removed: "embdes CAN-HCV 1.3"
