File: hardware/HCV.kicad_sch (KiCad schematic)
At the start: 33 parts, among them J1 USB_B_Micro, J2 Conn_ARM_SWD_TagConnect_TC2030, J4 Conn_01x02, SW2 SW_DIP_x02, U1 ESP32-WROOM-32U, U2 TPS562242, U3 SN65HVD232, U4 ADuM1201AR

Commit message: Updated Docu, Updated Hardware
Parts:
- removed J1: USB_B_Micro, Connector_USB:USB_C_Receptacle_Palconn_UTC16-G, symbol Connector:USB_C_Receptacle_USB2.0_16P
- removed JP1, JP2: Jumper_2_Open, Jumper:SolderJumper-2_P1.3mm_Open_RoundedPad1.0x1.5mm, symbol Jumper:Jumper_2_Open
- removed R1, R2: 5R, Resistor_SMD:R_0805_2012Metric, symbol Device:R
- removed SW2: SW_DIP_x02, Package_DIP:DIP-4_W7.62mm, symbol Switch:SW_DIP_x02
- removed U3: SN65HVD232, Package_SO:SOIC-8_3.9x4.9mm_P1.27mm, symbol Interface_CAN_LIN:SN65HVD232
- added C11, C12: 100n, Capacitor_SMD:C_0603_1608Metric, symbol Device:C_Small
- added J3: USB_C_Receptacle_PowerOnly_6P, Connector_USB:USB_C_Receptacle_GCT_USB4125-xx-x-0190_6P_TopMnt_Horizontal, symbol Connector:USB_C_Receptacle_PowerOnly_6P
- added SW2: SW_DIP_x04, Package_DIP:DIP-8_W7.62mm, symbol Switch:SW_DIP_x04
- added U3: ATA6560, Package_SO:SOIC-8_3.9x4.9mm_P1.27mm, symbol Interface_CAN_LIN:SN65HVD230
- added U5: TEA1-0505, Converter_DCDC:Converter_DCDC_TRACO_TEA1-xxxx_THT, symbol Converter_DCDC:TEA1-0505
Connections:
- net GND: now also C11.2, J3.A12 (GND), J3.B12 (GND), J3.S1 (SHIELD), SW2.7, U5.1 (-Vin)
- net GNDA: now also C12.2, SW2.5, SW2.6, U3.2 (GND), U3.8 (STBY), U5.3 (-Vout)
- net OPTSW: now also SW2.2
- net at D3.1 (K), J4.1 (Pin_1): now also SW2.1, U3.7 (CANH)
- net at D4.1 (K), J4.2 (Pin_2), R7.2: now also U3.6 (CANL)
- net at U4.6 (VOB): now also U3.1 (D)
- net at U4.7 (VIA): now also U3.4 (R)
- net at R7.1: now also SW2.8
- net +12V renamed +5V
- net +5V: now also C11.1, J3.A9 (VBUS), J3.B9 (VBUS), U5.2 (+Vin)
- net +3.3VP renamed +5VP
- net +5VP: now also C12.1, U3.3 (VCC), U5.4 (+Vout)
- new net nRXONLY: SW2.3, U3.5 (NSIL)
- no-connect marks 34 -> 29
