File: hardware/HCV.kicad_sch (KiCad schematic)
At the start: 32 parts, among them J2 Conn_ARM_SWD_TagConnect_TC2030, J3 USB_C_Receptacle_PowerOnly_6P, J4 Conn_01x02, SW2 SW_DIP_x04, U1 ESP32-WROOM-32U, U2 TPS562242, U3 ATA6560, U4 ADuM1201AR, U5 TEA1-0505

Commit message: Update for HCV Hardware
Parts:
- removed C12: 100n, Capacitor_SMD:C_0603_1608Metric, symbol Device:C_Small
- removed D3, D4: 1N4148WT, Diode_SMD:D_SOD-523, symbol Diode:1N4148WT
- removed R7: 120R, Resistor_SMD:R_0805_2012Metric, symbol Device:R
- removed SW2: SW_DIP_x04, Package_DIP:DIP-8_W7.62mm, symbol Switch:SW_DIP_x04
- added C12: 33/16, Capacitor_Tantalum_SMD:CP_EIA-3528-12_Kemet-T, symbol Device:C_Polarized
- added C15: 100n, Capacitor_SMD:C_0603_1608Metric, symbol Device:C_Small
- added D3: PESD1CAN-UX, Package_TO_SOT_SMD:SOT-23-3, symbol pesd1can:PESD1CAN-UX
- added R1: 4k7, Resistor_SMD:R_0603_1608Metric, symbol Device:R
- added SW1: SW_Push, Button_Switch_SMD:SW_SPST_EVPBF, symbol Switch:SW_Push
- R8: value 520R -> 470R
Connections:
- net +5VP: now also C12.1, C15.2
- net GND: now also SW1.1
- net GNDA: now also C12.2, C15.1, D3.3 (C3), R1.1
- net nRXONLY: now also R1.2
- net at U1.16 (IO13): now also D1.1 (K); no longer R8.1
- net at U1.23 (IO15): now also R8.2; no longer D1.2 (A)
- net at U1.28 (IO17): now also SW1.2
- net at J4.1 (Pin_1), U3.7 (CANH): now also D3.1 (C1)
- net at J4.2 (Pin_2), U3.6 (CANL): now also D3.2 (C2)
- net OPTSW renamed CANR
- new net: D1.2 (A), R8.1
- no-connect marks 29 -> 27
Other:
- note added: "rt/gr"
- note removed: "green"
- moved on the sheet: D1
